File: PCB/PiedPiper.sch (EAGLE design)
At the start: 27 parts

Commit message: Added updated PCB
Parts:
- removed BIAS: (no value), pinhead:PINHD-1X2
- removed C5: 1u, rcl:C-USC0805
- removed RGAIN: (no value), rcl:R-US_R1206
- removed R_DIVIDE1, R_DIVIDE2: 10k, rcl:R-US_R1206
- removed TRIMCOMP, TRIMGAIN, TRIMNOISE, TRIMROT: (no value), rcl:R-TRIMM64W
- added 12V-5V: TSR_1-2450, TSR_1-2450:TSR_1-2450
- added GAIN, NOISE, ROT, T_COMP: JST-XH-02-PIN-LONG-PAD, Rembrandt Electronics - JST XH Connectors v1-0:JST-XH-02-PIN-LONG-PAD
- added S2: (no value), switch-dil:DP03
- MIC: value (none) -> JST-XH-02-PIN-LONG-PAD; device pinhead:PINHD-1X2 -> Rembrandt Electronics - JST XH Connectors v1-0:JST-XH-02-PIN-LONG-PAD
- renumbered MAX97_INPUT to MAX97_AMPLIFIER
Connections:
- removed net 3V: FEATHER.2, R_DIVIDE1.1
- removed net BIAS: BIAS.1, C5.1, R_DIVIDE1.2, R_DIVIDE2.1
- removed net SCL_5V0: MAX97_AMPLIFIER.5
- removed net SDA_5V0: MAX97_AMPLIFIER.4
- removed net VDDIO: MAX97_AMPLIFIER.6
- new net N$1: FEATHER2.8, S2.5
- new net N$3: FEATHER2.9, S2.6
- new net N$4: FEATHER2.4, S2.4
- new net SCL: FEATHER2.11, MAX97_AMPLIFIER.5
- new net SDA: FEATHER2.12, MAX97_AMPLIFIER.4
- net A2: no longer BIAS.2
- net AUD1: now also SHIFT_REGISTER.D0; no longer SHIFT_REGISTER.D3
- net AUD2: now also SHIFT_REGISTER.D7; no longer SHIFT_REGISTER.D2
- net AUD4: now also SHIFT_REGISTER.D6; no longer SHIFT_REGISTER.D0
- net AUD5: now also SHIFT_REGISTER.D5; no longer SHIFT_REGISTER.D7
- net AUD6: now also SHIFT_REGISTER.D2; no longer SHIFT_REGISTER.D5
- net AUD7: now also SHIFT_REGISTER.D4; no longer SHIFT_REGISTER.D6
- net AUD8: now also SHIFT_REGISTER.D3; no longer SHIFT_REGISTER.D4
- net AUDIOIN: now also MIC-2.S; no longer MIC.1
- net CLOCK: now also FEATHER2.6, SHIFT_REGISTER.SRCK; no longer FEATHER2.5, SHIFT_REGISTER.RCK
- net COMP: now also T_COMP-2.S; no longer TRIMCOMP.A
- net GAIN: now also GAIN-2.S; no longer RGAIN.2, TRIMGAIN.A
- net GND: now also 12V-5V.GND, GAIN-1.S, MIC-1.S, S2.1, S2.2, S2.3, T_COMP-1.S; no longer C5.2, MIC.2, RGAIN.1, R_DIVIDE2.2, TRIMCOMP.S, TRIMGAIN.S
- net LATCH: now also FEATHER2.7, SHIFT_REGISTER.RCK; no longer FEATHER2.6, SHIFT_REGISTER.SRCK
- net NOISE: now also NOISE-2.S; no longer TRIMNOISE.S
- net ROT: now also ROT-2.S; no longer TRIMROT.S
- net SER_IN: now also FEATHER2.5; no longer FEATHER2.7
- net SHDN_5V: now also FEATHER2.10
- net USB: now also 12V-5V.+VOUT, MAX97_AMPLIFIER.6, NOISE-1.S, ROT-1.S; no longer TRIMNOISE.A, TRIMROT.A
- net VDD: now also 12V-5V.+VIN
Other:
- moved on the sheet: COMP
